File: MORI_ICHI.kicad_sch (KiCad schematic)
At the start: 68 parts, among them J1 Power, J2 Digital/PWM, J3 Analog, J4 Digital/PWM, J5 KH-TYPE-C-16P, J6 Grove, J7 MJ-179PH, J8 FH-1x3SG/RH, J9 Conn_01x04, Q1 L8050QLT1G, Q2 L8050QLT1G, SW1 TS-1187A-B-A-B, SW2 TS-1187A-B-A-B, U1 ESP32-S3-WROOM-1-N16R8, U2 CP2102N-A02-GQFN28R, U3 L7805CDT-TR, U4 SGM2212-3.3XKC3G/TR, U5 74HCT14PW,118

Commit message: 回路図を公開用に整理
回路図を公開用に整理
Other:
- note added: "ESP32-S3-WROOM-1-N16R8"
- note added: "I2C拡張コネクタ部"
- note added: "NeoPixel回路 3.3V→5V変換部"
- note added: "UNOシールドピンソケット部"
- note added: "USB → UART 変換部"
- note added: "USBコネクタ部"
- note added: "リセット、ブートスイッチ部"
- note added: "電源LED"
- note added: "電源部"
- note removed: "NeoPixel回路へ3.3V→5V変換"
- title: ESP32-S3 WROOM DevKit-ICHI -> Forest Design ESP32-S3 WROOM DevKit-ICHI
- moved on the sheet: C1, C10, C11, C12, C13, C14, C2, C3, C4, C5, C6, C7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
